Commit message: Hidden Motors Turned Off

File: gym_pybullet_drones/assets/cf2xCable.urdf (robot description, URDF)
Before this commit: robot cf2, 10 links, 9 joints
Links:
- link cable_link: mass .1 -> 0
- link payload_link: mass .1 -> 0.2
- link tinysphere1: mass .1 -> 0
- link tinysphere2: mass .1 -> 0

Commit message: Modified to test controller with CABLE drone model

File: gym_pybullet_drones/assets/cf2xCable.urdf (robot description, URDF)
Before this commit: robot cf2, 10 links, 9 joints
Links:
- link payload_link: mass 0.2 -> 0.1

Commit message: Can Move Quadcopter

File: gym_pybullet_drones/assets/cf2xCable.urdf (robot description, URDF)
Before this commit: robot cf2, 10 links, 9 joints
Links:
- link payload_link: mass 0.1 -> 0

Commit message: increased mass, thrust, and started load slightly tilted. Also passed along angle of the rope

File: gym_pybullet_drones/assets/cf2xCable.urdf (robot description, URDF)
Before this commit: robot cf2, 10 links, 9 joints
Links:
- link base_link: mass 0.027 -> 0.27
- link payload_link: mass 0 -> 0.15
